Commit message: Removed shoulders from URDF, set masses according to anthropometric data, disabled motors in collision script.

File: data/human_adult_scan.urdf (robot description, URDF)
Before this commit: robot human adult, 23 links, 22 joints
Links:
- removed link left_shoulder
- removed link right_shoulder
- link belly: mass 5.0001 -> 9.452
- link chest: mass 5.0001 -> 14.688
- link head: mass 5.0001 -> 4.005818
- link left_arm: mass 5.0001 -> 1.904
- link left_foot: mass 5.0001 -> 0.493
- link left_forearm: mass 5.0001 -> 1.088
- link left_hand: mass 5.0001 -> 0.408
- link left_leg: mass 5.0001 -> 6.8
- link left_shin: mass 5.0001 -> 3.162
- link left_sole: mass 5.0001 -> 0.32867
- link left_toes: mass 5.0001 -> 0.1643
- link pelvis: mass 5.0001 -> 9.656
- link right_arm: mass 5.0001 -> 1.904
- link right_foot: mass 5.0001 -> 0.493
- link right_forearm: mass 5.0001 -> 1.088
- link right_hand: mass 5.0001 -> 0.408
- link right_leg: mass 5.0001 -> 6.8
- link right_shin: mass 5.0001 -> 3.162
- link right_sole: mass 5.0001 -> 0.32867
- link right_toes: mass 5.0001 -> 0.1643
Joints:
- removed joint chest_to_left_shoulder
- removed joint chest_to_right_shoulder
- removed joint left_shoulder_to_left_arm
- removed joint right_shoulder_to_right_arm
- added joint chest_to_left_arm: type spherical, parent chest, child left_arm, origin xyz=0.1925 0.329 0
- added joint chest_to_right_arm: type spherical, parent chest, child right_arm, origin xyz=-0.1925 0.329 0
