Commit message: Added sub-partioned model to walk module and corrected mass mistake in urdfs

File: script/walk/man.urdf (robot description, URDF)
Before this commit: robot human adult, 21 links, 20 joints
Links:
- link neck: mass 5.0001 -> 1.50218

File: script/walk/man_x_partitioned.urdf (robot description, URDF)
Before this commit: robot human adult, 21 links, 20 joints
Links:
- added link belly_back, mass 4.726; collision mesh filename=belly_2xback.stl scale=1 1 1
- added link chest_back, mass 7.344; collision mesh filename=chest_2xback.stl scale=1 1 1
- added link head_back, mass 2.670545333333333; collision mesh filename=head_3xback.stl scale=1 1 1
- added link neck_back, mass 0.75109; collision mesh filename=neckxback.stl scale=1 1 1
- added link pelvis_back, mass 4.828; collision mesh filename=pelvisxback.stl scale=1 1 1
- link belly: mass 9.452 -> 4.726; geometry collision mesh filename=belly_2xfront.stl scale=1 1 1
- link chest: mass 14.688 -> 7.344; geometry collision mesh filename=chest_2xfront.stl scale=1 1 1
- link head: mass 4.005818 -> 1.3352726666666666; geometry collision mesh filename=head_3xfront.stl scale=1 1 1
- link neck: mass 1.50218 -> 0.75109; geometry collision mesh filename=neckxfront.stl scale=1 1 1
- link pelvis: mass 9.656 -> 4.828; geometry collision mesh filename=pelvisxfront.stl scale=1 1 1
Joints:
- added joint belly_to_belly_back: type fixed, parent belly, child belly_back, origin xyz=0 0 0
- added joint chest_to_chest_back: type fixed, parent chest, child chest_back, origin xyz=0 0 0
- added joint head_to_head_back: type fixed, parent head, child head_back, origin xyz=0 0 0
- added joint neck_to_neck_back: type fixed, parent neck, child neck_back, origin xyz=0 0 0
- added joint pelvis_to_pelvis_back: type fixed, parent pelvis, child pelvis_back, origin xyz=0 0 0
