Commit message: xacro: bug fix

File: src/walker/child/child.urdf (robot description, URDF)
Before this commit: robot child, 21 links, 20 joints
Joints:
- joint belly_to_pelvis: origin xyz=[0, -0.05044751612903226, 0] -> xyz=0 -0.050447516129 0
- joint chest_to_belly: origin xyz=[0, 0, 0] -> xyz=0 0 0
- joint chest_to_left_arm: origin xyz=[0.0924871129032258, 0.15806888387096776, 0] -> xyz=0.0924871129032 0.158068883871 0
- joint chest_to_neck: origin xyz=[0, 0.1765663064516129, 0] -> xyz=0 0.176566306452 0
- joint chest_to_right_arm: origin xyz=[-0.0924871129032258, 0.15806888387096776, 0] -> xyz=-0.0924871129032 0.158068883871 0
- joint left_arm_to_left_forearm: origin xyz=[0, -0.179164, 0] -> xyz=0 -0.179164 0
- joint left_foot_to_left_sole: origin xyz=[0, -0.03301215243902438, 0.01692930894308943] -> xyz=0 -0.033012152439 0.0169293089431
- joint left_forearm_to_left_hand: origin xyz=[0, -0.13818499999999997, 0] -> xyz=0 -0.138185 0
- joint left_leg_to_left_shin: origin xyz=[0, -0.22586099999999998, 0] -> xyz=0 -0.225861 0
- joint left_shin_to_left_foot: origin xyz=[0, -0.20823049999999999, 0] -> xyz=0 -0.2082305 0
- joint left_sole_to_left_toes: origin xyz=[0, 0, 0.040630341463414626] -> xyz=0 0 0.0406303414634
- joint neck_to_head: origin xyz=[0, 0.028589999999999997, 0] -> xyz=0 0.02859 0
- joint pelvis_to_left_leg: origin xyz=[0.043721180645161284, -0.03363167741935484, 0] -> xyz=0.0437211806452 -0.0336316774194 0
- joint pelvis_to_right_leg: origin xyz=[-0.043721180645161284, -0.03363167741935484, 0] -> xyz=-0.0437211806452 -0.0336316774194 0
- joint right_arm_to_right_forearm: origin xyz=[0, -0.179164, 0] -> xyz=0 -0.179164 0
- joint right_foot_to_right_sole: origin xyz=[0, -0.03301215243902438, 0.01692930894308943] -> xyz=0 -0.033012152439 0.0169293089431
- joint right_forearm_to_right_hand: origin xyz=[0, -0.13818499999999997, 0] -> xyz=0 -0.138185 0
- joint right_leg_to_right_shin: origin xyz=[0, -0.22586099999999998, 0] -> xyz=0 -0.225861 0
- joint right_shin_to_right_foot: origin xyz=[0, -0.20823049999999999, 0] -> xyz=0 -0.2082305 0
- joint right_sole_to_right_toes: origin xyz=[0, 0, 0.040630341463414626] -> xyz=0 0 0.0406303414634

File: src/walker/child/xacro/length_ratio.xacro (robot description, xacro)
@@ -29,22 +29,7 @@
     <!-- * Scales stl files for desired ratios                                          -->
     <!-- * Scales connection points for desired ratios                                  -->
-    <!--  -->
     <!-- ============================================================================== -->
     <!--    Scale stl files                                                             -->
     <!-- ============================================================================== -->
-    <xacro:macro name="read_stl_file" params="filename scale">
-        <visual>
-            <geometry>
-                <mesh filename="${filename}" scale="${scale} ${scale} ${scale}"/>
-            </geometry>
-            <origin rpy="0 0 0" xyz="0 0 0"/>
-        </visual>
-        <collision>
-            <geometry>
-                <mesh filename="${filename}" scale="${scale} ${scale} ${scale}"/>
-            </geometry>
-            <origin rpy="0 0 0" xyz="0 0 0"/>
-        </collision>
-    </xacro:macro>
     <xacro:property name="stl_scale_chest"  value="${(chest_ratio * height)  / (1.75 * 0.21)}" />
     <xacro:property name="stl_scale_belly"  value="${(belly_ratio * height)  / (1.75 * 0.06)}" />

Commit message: corrected ratios

File: src/walker/child/child.urdf (robot description, URDF)
Before this commit: robot child, 21 links, 20 joints
Links:
- link head: geometry collision mesh filename=stl/head.stl scale=0.849191071429 0.849191071429 0.849191071429; visual mesh filename=stl/head.stl scale=0.849191071429 0.849191071429 0.849191071429
- link left_sole: geometry collision mesh filename=stl/sole_left.stl scale=0.483694541231 0.483694541231 0.483694541231; visual mesh filename=stl/sole_left.stl scale=0.483694541231 0.483694541231 0.483694541231
- link left_toes: geometry collision mesh filename=stl/toes_left.stl scale=0.483694541231 0.483694541231 0.483694541231; visual mesh filename=stl/toes_left.stl scale=0.483694541231 0.483694541231 0.483694541231
- link neck: geometry collision mesh filename=stl/neck.stl scale=0.849191071429 0.849191071429 0.849191071429; visual mesh filename=stl/neck.stl scale=0.849191071429 0.849191071429 0.849191071429
- link right_sole: geometry collision mesh filename=stl/sole_right.stl scale=0.483694541231 0.483694541231 0.483694541231; visual mesh filename=stl/sole_right.stl scale=0.483694541231 0.483694541231 0.483694541231
- link right_toes: geometry collision mesh filename=stl/toes_right.stl scale=0.483694541231 0.483694541231 0.483694541231; visual mesh filename=stl/toes_right.stl scale=0.483694541231 0.483694541231 0.483694541231
Joints:
- joint neck_to_head: origin xyz=0 0.02859 0 -> xyz=0 0.04458253125 0

File: src/walker/child/xacro/length_ratio.xacro (robot description, xacro)
@@ -13,6 +13,6 @@
     <xacro:property name="pelvis_width_ratio" value="${pelvis_ratio * 0.052/0.04}" />
     <!-- Head + Neck -->
-    <xacro:property name="neck_ratio" value="0.03" />
-    <xacro:property name="head_ratio" value="${head_neck_ratio - neck_ratio}" />
+    <xacro:property name="neck_ratio" value="${head_neck_ratio * 0.03/0.16}" />
+    <xacro:property name="head_ratio" value="${head_neck_ratio * 0.13/0.16}" />
     <!-- Arm -->
     <xacro:property name="arm_ratio"     value="0.188" />
@@ -43,6 +43,6 @@
     <xacro:property name="stl_scale_shin" value="${(shin_ratio * height) / (1.75 * 0.246)}" />
     <xacro:property name="stl_scale_foot" value="${(foot_ratio * height) / (1.75 * 0.039)}" />
-    <xacro:property name="stl_scale_sole" value="${(sole_ratio * height) / (1.75 * 0.020)}" />
-    <xacro:property name="stl_scale_toes" value="${(toe_ratio  * height) / (1.75 * 0.048)}" />
+    <xacro:property name="stl_scale_sole" value="${(sole_ratio * height) / (1.75 * 0.048)}" />
+    <xacro:property name="stl_scale_toes" value="${(toe_ratio  * height) / (1.75 * 0.024)}" />
     <!-- ============================================================================== -->
     <!--    Scale connection points (as [x, y, z])                                      -->

Commit message: arm scaling based on torso ratio

File: src/walker/child/child.urdf (robot description, URDF)
Before this commit: robot child, 21 links, 20 joints
Links:
- link left_arm: geometry collision mesh filename=stl/arm_left.stl scale=0.480452534562 0.480452534562 0.480452534562; visual mesh filename=stl/arm_left.stl scale=0.480452534562 0.480452534562 0.480452534562
- link left_forearm: geometry collision mesh filename=stl/arm_lower_left.stl scale=0.480452534562 0.480452534562 0.480452534562; visual mesh filename=stl/arm_lower_left.stl scale=0.480452534562 0.480452534562 0.480452534562
- link left_hand: geometry collision mesh filename=stl/hand_left.stl scale=0.480452534562 0.480452534562 0.480452534562; visual mesh filename=stl/hand_left.stl scale=0.480452534562 0.480452534562 0.480452534562
- link right_arm: geometry collision mesh filename=stl/arm_right.stl scale=0.480452534562 0.480452534562 0.480452534562; visual mesh filename=stl/arm_right.stl scale=0.480452534562 0.480452534562 0.480452534562
- link right_forearm: geometry collision mesh filename=stl/arm_lower_right.stl scale=0.480452534562 0.480452534562 0.480452534562; visual mesh filename=stl/arm_lower_right.stl scale=0.480452534562 0.480452534562 0.480452534562
- link right_hand: geometry collision mesh filename=stl/hand_right.stl scale=0.480452534562 0.480452534562 0.480452534562; visual mesh filename=stl/hand_right.stl scale=0.480452534562 0.480452534562 0.480452534562
Joints:
- joint left_arm_to_left_forearm: origin xyz=0 -0.179164 0 -> xyz=0 -0.158068883871 0
- joint left_forearm_to_left_hand: origin xyz=0 -0.138185 0 -> xyz=0 -0.121914830645 0
- joint right_arm_to_right_forearm: origin xyz=0 -0.179164 0 -> xyz=0 -0.158068883871 0
- joint right_forearm_to_right_hand: origin xyz=0 -0.138185 0 -> xyz=0 -0.121914830645 0

File: src/walker/child/xacro/length_ratio.xacro (robot description, xacro)
@@ -16,7 +16,7 @@
     <xacro:property name="head_ratio" value="${head_neck_ratio * 0.13/0.16}" />
     <!-- Arm -->
-    <xacro:property name="arm_ratio"     value="0.188" />
-    <xacro:property name="forearm_ratio" value="0.145" />
-    <xacro:property name="hand_ratio"    value="0.108" />
+    <xacro:property name="arm_ratio"     value="${0.188/0.31 * torso_ratio}" />
+    <xacro:property name="forearm_ratio" value="${0.145/0.31 * torso_ratio}" />
+    <xacro:property name="hand_ratio"    value="${0.108/0.31 * torso_ratio}" />
     <!-- Foot -->
     <xacro:property name="foot_ratio"       value="${shin_ratio * 0.039/0.246}" />

Commit message: neck ratio based on torso ratio

File: src/walker/child/child.urdf (robot description, URDF)
Before this commit: robot child, 21 links, 20 joints
Links:
- link head: geometry collision mesh filename=stl/head.stl scale=0.934284579936 0.934284579936 0.934284579936; visual mesh filename=stl/head.stl scale=0.934284579936 0.934284579936 0.934284579936
- link neck: geometry collision mesh filename=stl/neck.stl scale=0.480452534562 0.480452534562 0.480452534562; visual mesh filename=stl/neck.stl scale=0.480452534562 0.480452534562 0.480452534562
Joints:
- joint neck_to_head: origin xyz=0 0.04458253125 0 -> xyz=0 0.0252237580645 0

File: src/walker/child/xacro/length_ratio.xacro (robot description, xacro)
@@ -13,6 +13,6 @@
     <xacro:property name="pelvis_width_ratio" value="${pelvis_ratio * 0.052/0.04}" />
     <!-- Head + Neck -->
-    <xacro:property name="neck_ratio" value="${head_neck_ratio * 0.03/0.16}" />
-    <xacro:property name="head_ratio" value="${head_neck_ratio * 0.13/0.16}" />
+    <xacro:property name="neck_ratio" value="${0.03/0.31 * torso_ratio}" />
+    <xacro:property name="head_ratio" value="${head_neck_ratio - neck_ratio}" />
     <!-- Arm -->
     <xacro:property name="arm_ratio"     value="${0.188/0.31 * torso_ratio}" />

Commit message: Improvment in child head

File: src/walker/child/child.urdf (robot description, URDF)
Before this commit: robot child, 21 links, 20 joints
Links:
- link head: geometry collision mesh filename=stl/head_child.stl scale=0.878989634881 0.878989634881 0.48; visual mesh filename=stl/head_child.stl scale=0.878989634881 0.878989634881 0.48

File: src/walker/child/xacro/length_ratio.xacro (robot description, xacro)
@@ -4,5 +4,5 @@
     <xacro:property name="shin_ratio" value="0.2185" />
     <xacro:property name="torso_ratio" value="0.2735" />
-    <xacro:property name="head_neck_ratio" value="0.2495" />
+    <xacro:property name="head_neck_ratio" value="0.2363" />
     <!-- Torso = Chest + Belly + Pelvis -->
     <xacro:property name="chest_arm_ratio" value="${0.188/0.31 * torso_ratio}" />

Commit message: new head stl for child

File: src/walker/child/child.urdf (robot description, URDF)
Before this commit: robot child, 21 links, 20 joints
Links:
- link head: geometry collision mesh filename=stl/head_child.stl scale=0.878989634881 0.878989634881 0.878989634881; visual mesh filename=stl/head_child.stl scale=0.878989634881 0.878989634881 0.878989634881

File: src/walker/child/xacro/macros.xacro (robot description, xacro)
@@ -4,10 +4,15 @@
         <origin xyz="${conn_name[0]} ${conn_name[1]} ${conn_name[2]}"/>
     </xacro:macro>
-    <xacro:macro name="read_stl_file" params="filename scale">
+    <xacro:macro name="read_stl_file"
+                 params="filename
+                         scale
+                         xyz:=${list([0,0,0])}
+                         rpy:=${list([0,0,0])}">
         <visual>
             <geometry>
                 <mesh filename="${filename}" scale="${scale} ${scale} ${scale}"/>
             </geometry>
-            <origin rpy="0 0 0" xyz="0 0 0"/>
+            <origin rpy="${rpy[0]} ${rpy[1]} ${rpy[2]}"
+                    xyz="${xyz[0]} ${xyz[1]} ${xyz[2]}"/>
         </visual>
         <collision>
@@ -15,5 +20,6 @@
                 <mesh filename="${filename}" scale="${scale} ${scale} ${scale}"/>
             </geometry>
-            <origin rpy="0 0 0" xyz="0 0 0"/>
+            <origin rpy="${rpy[0]} ${rpy[1]} ${rpy[2]}"
+                    xyz="${xyz[0]} ${xyz[1]} ${xyz[2]}"/>
         </collision>
     </xacro:macro>

Commit message: updated child local proportions

File: src/walker/child/child.urdf (robot description, URDF)
Before this commit: robot child, 21 links, 20 joints
Links:
- link head: geometry collision mesh filename=stl/head_child.stl scale=0.878989634881 0.878989634881 0.878989634881; visual mesh filename=stl/head_child.stl scale=0.597608321217 0.878989634881 0.652486485509
- link neck: geometry collision mesh filename=stl/neck.stl scale=0.480452534562 0.480452534562 0.480452534562; visual mesh filename=stl/neck.stl scale=0.534976171601 0.480452534562 0.513688128009

File: src/walker/child/xacro/length_ratio.xacro (robot description, xacro)
@@ -25,8 +25,14 @@
     <xacro:property name="toe_ratio"  value="${sole_ratio / 2}" />
     <!-- ============================================================================== -->
+    <!--    Child local proportions                                                     -->
+    <!-- ============================================================================== -->
+    <xacro:property name="local_neck" value="${[3.0711/2.7581, 1, 3.0711/2.8724]}" />
+    <xacro:property name="local_head" value="${[0.6397/0.9409, 1, 0.7461/1.0051]}" />
+    <!-- ============================================================================== -->
     <!-- ========================= DO NOT CHANGE AFTER THIS LINE ====================== -->
     <!-- ============================================================================== -->
     <!-- * Scales stl files for desired ratios                                          -->
     <!-- * Scales connection points for desired ratios                                  -->
+    <!--  -->
     <!-- ============================================================================== -->
     <!--    Scale stl files                                                             -->

File: src/walker/child/xacro/macros.xacro (robot description, xacro)
@@ -7,9 +7,11 @@
                  params="filename
                          scale
+                         local_proportion:=${list([1,1,1])}
                          xyz:=${list([0,0,0])}
                          rpy:=${list([0,0,0])}">
         <visual>
             <geometry>
-                <mesh filename="${filename}" scale="${scale} ${scale} ${scale}"/>
+                <mesh filename="${filename}"
+                      scale="${scale*local_proportion[0]} ${scale*local_proportion[1]} ${scale*local_proportion[2]}"/>
             </geometry>
             <origin rpy="${rpy[0]} ${rpy[1]} ${rpy[2]}"
