Commit message: + changed child head

File: src/human/child/child.urdf (robot description, URDF)
Before this commit: robot child, 21 links, 20 joints
Links:
- link head: geometry collision mesh filename=stl/head_child.stl scale=0.878989634881 0.878989634881 0.878989634881; visual mesh filename=stl/head_child.stl scale=0.878989634881 0.878989634881 0.878989634881

File: src/human/child/xacro/length_ratio.xacro (robot description, xacro)
@@ -28,5 +28,5 @@
     <!-- ============================================================================== -->
     <xacro:property name="local_neck" value="${[3.0711/2.7581, 1, 3.0711/2.8724]}" />
-    <xacro:property name="local_head" value="${[0.6397/0.9409, 1, 0.7461/1.0051]}" />
+    <xacro:property name="local_head" value="${[1, 1, 1]}" />
     <!-- ============================================================================== -->
     <!-- ========================= DO NOT CHANGE AFTER THIS LINE ====================== -->

File: src/human/child/xacro/mass_ratio.xacro (robot description, xacro)
@@ -3,5 +3,5 @@
     The segment mass data is calculated using the table 4.1 from the book.
     This model's additional details (feet), which are implemented here, are given in
-        Terlemez, Ö., Ulbrich, S., Mandery, C., Do, M., Vahrenkamp, N., & Asfour, T. (2014, November).
+        Terlemez, O., Ulbrich, S., Mandery, C., Do, M., Vahrenkamp, N., & Asfour, T. (2014, November).
         "Master Motor Map (MMM)—Framework and toolkit for capturing, representing, and reproducing human
         motion on humanoid robots", in 2014 IEEE-RAS International Conference on Humanoid Robots (pp. 894-901)
