Commit message: Add files via upload

File: src/robot/starship/starship_full_load.urdf (robot description, URDF)
Before this commit: robot starship, 2 links, 1 joints
Links:
- link starship_main: geometry collision mesh filename=stl/starship.stl scale=0.001 0.001 0.001; visual mesh filename=stl/starship.stl scale=0.001 0.001 0.001
